File: BPF.sch (KiCad schematic (older format))
At the start: 36 parts, among them J6 Conn_Coaxial, K1 FRT5, K4 FRT5, Q4 MMBT2222LT1G

Commit message: production
Connections:
- net OUT: now reaches J6.1 (In), K1.3
Changed lines of the file:
@@
 Text GLabel 10350 1750 2    60   Input ~ 0
 BAND
+Wire Wire Line
+	1450 2600 1450 2500
+Connection ~ 1450 2600
+Text GLabel 1450 2500 1    60   BiDi ~ 0
+OUT
 $EndSCHEMATC
