File: LCSDR.sch (KiCad schematic (older format))
At the start: 8 parts, among them J1 Conn_01x10, J10 Conn_01x01, J11 Conn_01x01, J2 Conn_01x10, J5 Conn_01x10, J8 Conn_01x01, J9 Conn_01x01

Commit message: first edit
Changed lines of the file:
@@
 S 3600 2700 2600 1700
 U 5DC357A0
-F0 "AUDIO_OUT" 60
-F1 "AUDIO_OUT.sch" 60
+F0 "s1" 60
+F1 "s1.sch" 60
 $EndSheet
 $Sheet
@@
 $EndComp
 $Comp
-L GND #PWR7
+L GND #PWR01
 U 1 1 5DE25560
 P 9550 6300
-F 0 "#PWR7" H 9550 6050 50  0001 C CNN
+F 0 "#PWR01" H 9550 6050 50  0001 C CNN
 F 1 "GND" H 9550 6150 50  0000 C CNN
 F 2 "" H 9550 6300 50  0001 C CNN
@@
 $EndComp
 $Comp
-L GND #PWR8
+L GND #PWR02
 U 1 1 5DE25589
 P 9900 6300
-F 0 "#PWR8" H 9900 6050 50  0001 C CNN
+F 0 "#PWR02" H 9900 6050 50  0001 C CNN
 F 1 "GND" H 9900 6150 50  0000 C CNN
 F 2 "" H 9900 6300 50  0001 C CNN
@@
 $EndComp
 $Comp
-L GND #PWR9
+L GND #PWR03
 U 1 1 5DE255A6
 P 10250 6300
-F 0 "#PWR9" H 10250 6050 50  0001 C CNN
+F 0 "#PWR03" H 10250 6050 50  0001 C CNN
 F 1 "GND" H 10250 6150 50  0000 C CNN
 F 2 "" H 10250 6300 50  0001 C CNN
@@
 $EndComp
 $Comp
-L GND #PWR10
+L GND #PWR04
 U 1 1 5DE255C3
 P 10600 6300
-F 0 "#PWR10" H 10600 6050 50  0001 C CNN
+F 0 "#PWR04" H 10600 6050 50  0001 C CNN
 F 1 "GND" H 10600 6150 50  0000 C CNN
 F 2 "" H 10600 6300 50  0001 C CNN
@@
 S 3600 4650 2600 1700
 U 5DE7E102
-F0 "switching" 60
-F1 "switching.sch" 60
+F0 "s2" 60
+F1 "s2.sch" 60
 $EndSheet
 $Sheet
@@
 S 5200 750  2000 1100
 U 5EA97077
-F0 "MIXERS" 60
-F1 "MIXERS.sch" 60
+F0 "MIXER" 60
+F1 "MIXER.sch" 60
 $EndSheet
 Text GLabel 9700 750  0    60   Input ~ 0
@@
 	7300 5400 8200 5400
 $Comp
-L GND #PWR2
+L GND #PWR05
 U 1 1 5EAD338C
 P 8100 5300
-F 0 "#PWR2" H 8100 5050 50  0001 C CNN
+F 0 "#PWR05" H 8100 5050 50  0001 C CNN
 F 1 "GND" H 8100 5150 50  0001 C CNN
 F 2 "" H 8100 5300 50  0001 C CNN
@@
 	7300 5800 8200 5800
 $Comp
-L GND #PWR3
+L GND #PWR06
 U 1 1 5EAD4510
 P 8100 5500
-F 0 "#PWR3" H 8100 5250 50  0001 C CNN
+F 0 "#PWR06" H 8100 5250 50  0001 C CNN
 F 1 "GND" H 8100 5350 50  0001 C CNN
 F 2 "" H 8100 5500 50  0001 C CNN
@@
 	8100 5500 8200 5500
 $Comp
-L GND #PWR4
+L GND #PWR07
 U 1 1 5EAD456B
 P 8100 5700
-F 0 "#PWR4" H 8100 5450 50  0001 C CNN
+F 0 "#PWR07" H 8100 5450 50  0001 C CNN
 F 1 "GND" H 8100 5550 50  0001 C CNN
 F 2 "" H 8100 5700 50  0001 C CNN
@@
 	8150 1500 8400 1500
 $Comp
-L GND #PWR6
+L GND #PWR08
 U 1 1 5EAE9B68
 P 8300 1400
-F 0 "#PWR6" H 8300 1150 50  0001 C CNN
+F 0 "#PWR08" H 8300 1150 50  0001 C CNN
 F 1 "GND" H 8300 1250 50  0001 C CNN
 F 2 "" H 8300 1400 50  0001 C CNN
@@
 $EndComp
 $Comp
-L GND #PWR1
+L GND #PWR09
 U 1 1 5EAECBA9
 P 8100 5100
-F 0 "#PWR1" H 8100 4850 50  0001 C CNN
+F 0 "#PWR09" H 8100 4850 50  0001 C CNN
 F 1 "GND" H 8100 4950 50  0001 C CNN
 F 2 "" H 8100 5100 50  0001 C CNN
@@
 	8100 5100 8200 5100
 $Comp
-L GND #PWR5
+L GND #PWR010
 U 1 1 5EAECD33
 P 8100 5900
-F 0 "#PWR5" H 8100 5650 50  0001 C CNN
+F 0 "#PWR010" H 8100 5650 50  0001 C CNN
 F 1 "GND" H 8100 5750 50  0001 C CNN
 F 2 "" H 8100 5900 50  0001 C CNN

Commit message: need some GND vias
Parts:
- removed RN4: 47, Resistors_SMD:R_Array_Convex_4x0603, symbol R_Pack04
- added J7: Conn_01x10, Pin_Headers:Pin_Header_Straight_1x10_Pitch2.54mm, symbol Conn_01x10
- renumbered J2 to J1, J1 to J2
Connections:
- net labels added: +12V, +9V, BAND, BPF, IF_RX_TX, MIXER, PTT, ROTATE, S1_RX_TX, S2_RX_TX
- net labels removed: ADC, IO2, IO3, IO4, IO5, IO6, IO7, Voltage1, Voltage2, ~RX, ~TX
- wire segments 56 -> 39
Other:
- moved on the sheet: J1, J2

Commit message: production
Connections:
- net GND: now also J7.1 (Pin_1), J7.3 (Pin_3)
- net OUT: now reaches J7.2 (Pin_2)
Changed lines of the file:
@@
 	1    0    0    -1
 $EndComp
+Text GLabel 7950 3150 0    60   BiDi ~ 0
+OUT
+Wire Wire Line
+	7950 3150 8200 3150
+$Comp
+L GND #PWR?
+U 1 1 5EBCD351
+P 8100 4200
+F 0 "#PWR?" H 8100 3950 50  0001 C CNN
+F 1 "GND" H 8100 4050 50  0001 C CNN
+F 2 "" H 8100 4200 50  0001 C CNN
+F 3 "" H 8100 4200 50  0001 C CNN
+	1    8100 4200
+	1    0    0    -1
+$EndComp
+Wire Wire Line
+	8100 4200 8100 3050
+Wire Wire Line
+	8100 3050 8200 3050
+Wire Wire Line
+	8200 3250 8100 3250
+Connection ~ 8100 3250
 $EndSCHEMATC
