File: s2.sch (KiCad schematic (older format))
At the start: 63 parts, among them J3 phones, J4 MIC_PTT, Q1 2N7002, Q2 BC847, U6 NE5532, U8 4053, U9 4053

Commit message: first edit
Parts:
- removed C21: 22..47nF, UI:C_1206_0603, symbol C_Small
- removed C39: 10uF, Capacitors_THT:CP_Radial_D5.0mm_P2.00mm, symbol CP_Small
- removed C42: 100nF, UI:C_1206_0603, symbol C_Small
- removed C52, C53, C54, C55: 1uF, Capacitors_THT:CP_Radial_D5.0mm_P2.00mm, symbol CP_Small
- removed R17, R22, R23, R5, R6: 10k, UI:R_1206_0603, symbol R_Small
- removed U8, U9: 4053, Housings_SOIC:SOIC-16_3.9x9.9mm_Pitch1.27mm, symbol 4053
- added K2, K3: FRT5, Relays_THT:Relay_DPDT_FRT5, symbol FRT5
Connections:
- wire segments 144 -> 118
Other:
- moved on the sheet: C14, C15, C8

Commit message: rotators 2 74lvc1G74
Parts:
- removed C43, C56: 100nF, UI:C_1206_0603, symbol C_Small
- removed C48: 22..47nF, UI:C_1206_0603, symbol C_Small
- removed C57: 10uF, Capacitors_THT:CP_Radial_D5.0mm_P2.00mm, symbol CP_Small
- removed K2, K3: FRT5, Relays_THT:Relay_DPDT_FRT5, symbol FRT5
- removed Q1: 2N7002, TO_SOT_Packages_SMD:SOT-23, symbol Q_NMOS_GSD
- removed R26, R27: 10k, UI:R_1206_0603, symbol R_Small
- added C21: 100nF, UI:C_1206_0603, symbol C_Small
- added D1: LL4148, symbol D_Small
- added K2, K3: G6K-2F, UI:Relay_G6K-2F, symbol G6K-2F
- added Q1: MMBT2222LT1G, TO_SOT_Packages_SMD:SOT-23, symbol Q_NPN_BEC
- C12, C13, C27, C31: footprint UI:C_1206_0603 -> Capacitors_SMD:C_0603_HandSoldering
- C14, C8: value 1uF -> 4.7uF; footprint Capacitors_THT:CP_Radial_D5.0mm_P2.00mm -> Capacitors_Tantalum_SMD:CP_Tantalum_Case-A_EIA-3216-18_Wave
- C22, C23: footprint Capacitors_THT:CP_Radial_D5.0mm_P2.00mm -> Capacitors_Tantalum_SMD:CP_Tantalum_Case-A_EIA-3216-18_Wave
- L5, L6: footprint (none) -> Choke_Axial_ThroughHole:Choke_Horizontal_RM10mm
- R24, R25, R30, R31, R33, R34: footprint UI:R_1206_0603 -> Resistors_SMD:R_0603_HandSoldering
Connections:
- net labels added: +12V
- net labels removed: +9V, TX
- wire segments 118 -> 103
Other:
- moved on the sheet: C14, C51, C8, R18

Commit message: PCB s1
Parts:
- C15, C16: footprint Capacitors_THT:CP_Radial_D5.0mm_P2.00mm -> Capacitors_Tantalum_SMD:CP_Tantalum_Case-A_EIA-3216-18_Wave
Changed lines of the file:
@@
 Q_IN
 $Comp
-L GND #PWR42
+L GND #PWR025
 U 1 1 5DE7E3AF
 P 8050 4400
-F 0 "#PWR42" H 8050 4150 50  0001 C CNN
+F 0 "#PWR025" H 8050 4150 50  0001 C CNN
 F 1 "GND" H 8050 4250 50  0001 C CNN
 F 2 "" H 8050 4400 50  0001 C CNN
@@
 $EndComp
 $Comp
-L GND #PWR43
+L GND #PWR026
 U 1 1 5DE7E3B9
 P 8350 3900
-F 0 "#PWR43" H 8350 3650 50  0001 C CNN
+F 0 "#PWR026" H 8350 3650 50  0001 C CNN
 F 1 "GND" H 8350 3750 50  0001 C CNN
 F 2 "" H 8350 3900 50  0001 C CNN
@@
 $EndComp
 $Comp
-L GND #PWR44
+L GND #PWR027
 U 1 1 5DE7E3DB
 P 8450 4500
-F 0 "#PWR44" H 8450 4250 50  0001 C CNN
+F 0 "#PWR027" H 8450 4250 50  0001 C CNN
 F 1 "GND" H 8450 4350 50  0001 C CNN
 F 2 "" H 8450 4500 50  0001 C CNN
@@
 F 0 "C15" V 5700 1850 50  0000 L CNN
 F 1 "1uF" V 5600 1850 50  0000 L CNN
-F 2 "Capacitors_THT:CP_Radial_D5.0mm_P2.00mm" H 5800 1900 50  0001 C CNN
+F 2 "Capacitors_Tantalum_SMD:CP_Tantalum_Case-A_EIA-3216-18_Wave" H 5800 1900 50  0001 C CNN
 F 3 "" H 5800 1900 50  0001 C CNN
 	1    5800 1900
@@
 F 0 "C16" V 5450 1450 50  0000 L CNN
 F 1 "1uF" V 5350 1450 50  0000 L CNN
-F 2 "Capacitors_THT:CP_Radial_D5.0mm_P2.00mm" H 5250 1500 50  0001 C CNN
+F 2 "Capacitors_Tantalum_SMD:CP_Tantalum_Case-A_EIA-3216-18_Wave" H 5250 1500 50  0001 C CNN
 F 3 "" H 5250 1500 50  0001 C CNN
 	1    5250 1500
@@
 	4200 3050 4200 3150
 $Comp
-L GND #PWR36
+L GND #PWR028
 U 1 1 5EA8447C
 P 4200 3400
-F 0 "#PWR36" H 4200 3150 50  0001 C CNN
+F 0 "#PWR028" H 4200 3150 50  0001 C CNN
 F 1 "GND" H 4200 3250 50  0001 C CNN
 F 2 "" H 4200 3400 50  0001 C CNN
@@
 	3050 2550 3400 2550
 $Comp
-L GND #PWR34
+L GND #PWR029
 U 1 1 5EA86A3F
 P 3200 3000
-F 0 "#PWR34" H 3200 2750 50  0001 C CNN
+F 0 "#PWR029" H 3200 2750 50  0001 C CNN
 F 1 "GND" H 3200 2850 50  0001 C CNN
 F 2 "" H 3200 3000 50  0001 C CNN
@@
 Connection ~ 2700 2550
 $Comp
-L GND #PWR31
+L GND #PWR030
 U 1 1 5EA87223
 P 2700 3000
-F 0 "#PWR31" H 2700 2750 50  0001 C CNN
+F 0 "#PWR030" H 2700 2750 50  0001 C CNN
 F 1 "GND" H 2700 2850 50  0001 C CNN
 F 2 "" H 2700 3000 50  0001 C CNN
@@
 Connection ~ 2200 2650
 $Comp
-L GND #PWR26
+L GND #PWR031
 U 1 1 5EA87A28
 P 1500 2950
-F 0 "#PWR26" H 1500 2700 50  0001 C CNN
+F 0 "#PWR031" H 1500 2700 50  0001 C CNN
 F 1 "GND" H 1500 2800 50  0001 C CNN
 F 2 "" H 1500 2950 50  0001 C CNN
@@
 $EndComp
 $Comp
-L GND #PWR28
+L GND #PWR032
 U 1 1 5EA87D5A
 P 2200 3000
-F 0 "#PWR28" H 2200 2750 50  0001 C CNN
+F 0 "#PWR032" H 2200 2750 50  0001 C CNN
 F 1 "GND" H 2200 2850 50  0001 C CNN
 F 2 "" H 2200 3000 50  0001 C CNN
@@
 $EndComp
 $Comp
-L GND #PWR30
+L GND #PWR033
 U 1 1 5EA88DC1
 P 2700 1950
-F 0 "#PWR30" H 2700 1700 50  0001 C CNN
+F 0 "#PWR033" H 2700 1700 50  0001 C CNN
 F 1 "GND" H 2700 1800 50  0001 C CNN
 F 2 "" H 2700 1950 50  0001 C CNN
@@
 $EndComp
 $Comp
-L GND #PWR29
+L GND #PWR034
 U 1 1 5EA88EC8
 P 2700 1700
-F 0 "#PWR29" H 2700 1450 50  0001 C CNN
+F 0 "#PWR034" H 2700 1450 50  0001 C CNN
 F 1 "GND" H 2700 1550 50  0001 C CNN
 F 2 "" H 2700 1700 50  0001 C CNN
@@
 	2200 1350 2200 1200
 $Comp
-L GND #PWR27
+L GND #PWR035
 U 1 1 5EA8A2B0
 P 1850 1700
-F 0 "#PWR27" H 1850 1450 50  0001 C CNN
+F 0 "#PWR035" H 1850 1450 50  0001 C CNN
 F 1 "GND" H 1850 1550 50  0001 C CNN
 F 2 "" H 1850 1700 50  0001 C CNN
@@
 Connection ~ 3950 5400
 $Comp
-L GND #PWR35
+L GND #PWR036
 U 1 1 5EA8DADD
 P 3950 5700
-F 0 "#PWR35" H 3950 5450 50  0001 C CNN
+F 0 "#PWR036" H 3950 5450 50  0001 C CNN
 F 1 "GND" H 3950 5550 50  0001 C CNN
 F 2 "" H 3950 5700 50  0001 C CNN
@@
 $EndComp
 $Comp
-L GND #PWR38
+L GND #PWR037
 U 1 1 5EA9039E
 P 4300 5700
-F 0 "#PWR38" H 4300 5450 50  0001 C CNN
+F 0 "#PWR037" H 4300 5450 50  0001 C CNN
 F 1 "GND" H 4300 5550 50  0001 C CNN
 F 2 "" H 4300 5700 50  0001 C CNN
@@
 $EndComp
 $Comp
-L GND #PWR40
+L GND #PWR038
 U 1 1 5EA91527
 P 4750 5700
-F 0 "#PWR40" H 4750 5450 50  0001 C CNN
+F 0 "#PWR038" H 4750 5450 50  0001 C CNN
 F 1 "GND" H 4750 5550 50  0001 C CNN
 F 2 "" H 4750 5700 50  0001 C CNN
@@
 	1500 5800 1650 5800
 $Comp
-L GND #PWR32
+L GND #PWR039
 U 1 1 5EA93E43
 P 2800 5350
-F 0 "#PWR32" H 2800 5100 50  0001 C CNN
+F 0 "#PWR039" H 2800 5100 50  0001 C CNN
 F 1 "GND" H 2800 5200 50  0001 C CNN
 F 2 "" H 2800 5350 50  0001 C CNN
@@
 $EndComp
 $Comp
-L GND #PWR33
+L GND #PWR040
 U 1 1 5EA93F05
 P 2800 6900
-F 0 "#PWR33" H 2800 6650 50  0001 C CNN
+F 0 "#PWR040" H 2800 6650 50  0001 C CNN
 F 1 "GND" H 2800 6750 50  0001 C CNN
 F 2 "" H 2800 6900 50  0001 C CNN
@@
 $EndComp
 $Comp
-L GND #PWR25
+L GND #PWR041
 U 1 1 5EA94135
 P 850 5850
-F 0 "#PWR25" H 850 5600 50  0001 C CNN
+F 0 "#PWR041" H 850 5600 50  0001 C CNN
 F 1 "GND" H 850 5700 50  0001 C CNN
 F 2 "" H 850 5850 50  0001 C CNN
@@
 Connection ~ 4300 4450
 $Comp
-L GND #PWR37
+L GND #PWR042
 U 1 1 5EA94B85
 P 4300 4700
-F 0 "#PWR37" H 4300 4450 50  0001 C CNN
+F 0 "#PWR042" H 4300 4450 50  0001 C CNN
 F 1 "GND" H 4300 4550 50  0001 C CNN
 F 2 "" H 4300 4700 50  0001 C CNN
@@
 $EndComp
 $Comp
-L GND #PWR39
+L GND #PWR043
 U 1 1 5EA94C4D
 P 4750 4700
-F 0 "#PWR39" H 4750 4450 50  0001 C CNN
+F 0 "#PWR043" H 4750 4450 50  0001 C CNN
 F 1 "GND" H 4750 4550 50  0001 C CNN
 F 2 "" H 4750 4700 50  0001 C CNN
@@
 	7150 4650 7000 4650
 $Comp
-L +12V #PWR41
+L +12V #PWR044
 U 1 1 5EB0655B
 P 6350 4000
-F 0 "#PWR41" H 6350 3850 50  0001 C CNN
+F 0 "#PWR044" H 6350 3850 50  0001 C CNN
 F 1 "+12V" H 6350 4140 50  0000 C CNN
 F 2 "" H 6350 4000 50  0001 C CNN

Commit message: need some GND vias
Parts:
- removed K2, K3: G6K-2F, UI:Relay_G6K-2F, symbol G6K-2F
- added C69: 100nF, UI:C_1206_0603, symbol C_Small
- added D3: LL4148, Diodes_SMD:D_MiniMELF, symbol D_Small
- added K2, K3: FRT5, Relays_THT:Relay_DPDT_FRT5, symbol FRT5
- C11: value 3.3nF -> 1.5nF
- C12, C13: value 100nF -> 220pF; footprint Capacitors_SMD:C_0603_HandSoldering -> UI:C_1206_0603
- C14, C22, C23, C8: footprint Capacitors_Tantalum_SMD:CP_Tantalum_Case-A_EIA-3216-18_Wave -> Capacitors_THT:CP_Radial_D5.0mm_P2.00mm
- C27, C31: footprint Capacitors_SMD:C_0603_HandSoldering -> UI:C_1206_0603
- C51: footprint UI:C_1206_0603 -> Capacitors_SMD:C_0603_HandSoldering
- D1: footprint (none) -> Diodes_SMD:D_MiniMELF
- R24, R25, R33, R34: footprint Resistors_SMD:R_0603_HandSoldering -> UI:R_1206_0603
- R30, R31: value 10k -> 6.8k; footprint Resistors_SMD:R_0603_HandSoldering -> UI:R_1206_0603
Connections:
- net labels added: PTT, RX_9V, S2_RX_TX
- wire segments 103 -> 116
